Commit message: edit denso robot

File: urdf/denso060.urdf (robot description, URDF)
Before this commit: robot vs060, 8 links, 7 joints
Links:
- removed link J6
- removed link world_1
- added link BASE, mass 1000; collision mesh filename=package://denso060/BASE_mesh.stl; visual mesh filename=package://denso060/BASE_mesh.stl
- added link Flange, mass 4.154; collision mesh filename=package://denso060/Flange_mesh.stl; visual mesh filename=package://denso060/Flange_mesh.stl
- link J1: mass 1 -> 4.327; geometry collision mesh filename=package://denso060/J1_mesh.stl; visual mesh filename=package://denso060/J1_mesh.stl
- link J2: mass 1 -> 9.475; geometry collision mesh filename=package://denso060/J2_mesh.stl; visual mesh filename=package://denso060/J2_mesh.stl
- link J3: mass 1 -> 4.097; geometry collision mesh filename=package://denso060/J3_mesh.stl; visual mesh filename=package://denso060/J3_mesh.stl
- link J4: mass 1 -> 1.779; geometry collision mesh filename=package://denso060/J4_mesh.stl; visual mesh filename=package://denso060/J4_mesh.stl
- link J5: mass 1 -> 1.211; geometry collision mesh filename=package://denso060/J5_mesh.stl; visual mesh filename=package://denso060/J5_mesh.stl
- link base_link: mass 1 -> None; geometry 
Joints:
- removed joint joint_1
- removed joint joint_2
- removed joint joint_3
- removed joint joint_4
- removed joint joint_5
- removed joint joint_6
- removed joint joint_w
- added joint base_link_joint: type fixed, parent base_link, child BASE
- added joint flange: type revolute, parent J5, child Flange, origin xyz=0 1.55431e-17 0.07 rpy=0 -0 0 , axis 0 0 1, limit lower=-6.28319 upper=6.28319 effort=33.5103 velocity=0.5
- added joint j1: type revolute, parent BASE, child J1, origin xyz=0 4.04121e-17 0.182 rpy=0 -0 0 , axis 0 0 1, limit lower=-2.96706 upper=2.96706 effort=19.7336 velocity=0.5
- added joint j2: type revolute, parent J1, child J2, origin xyz=0 3.61933e-17 0.163 rpy=0 -0 0 , axis 0 1 0, limit lower=-2.0944 upper=2.0944 effort=16.8447 velocity=0.5
- added joint j3: type revolute, parent J2, child J3, origin xyz=0 6.77236e-17 0.305 rpy=0 -0 0 , axis 0 1 0, limit lower=-2.18166 upper=2.70526 effort=20.7089 velocity=0.5
- added joint j4: type revolute, parent J3, child J4, origin xyz=-0.01 3.66374e-17 0.165 rpy=0 -0 0 , axis 0 0 1, limit lower=-4.71239 upper=4.71239 effort=20.9665 velocity=0.5
- added joint j5: type revolute, parent J4, child J5, origin xyz=0 2.9976e-17 0.135 rpy=0 -0 0 , axis 0 1 0, limit lower=-2.0944 upper=2.0944 effort=23.7229 velocity=0.5

Commit message: fix mass

File: urdf/denso060.urdf (robot description, URDF)
Before this commit: robot vs060A1_AV6_NNN_NNN, 8 links, 7 joints
Links:
- link BASE: mass 1000 -> 10.00
